File: LEDBoard_4x4_16bit.sch (KiCad schematic (older format))
At the start: 35 parts, among them J1 signal_in, J2 power, J6 signal_out, U1 TLC5971RGER, U2 TLC5971RGER, U3 TLC5971RGER, U4 TLC5971RGER

Commit message: updated things
Parts:
- C1, C2, C3, C4: mouser (none) -> 81-GRM39X104K50D; murata (none) -> GRM188R71H104KA93D
- C5: value 47uF -> 47uF 6.3V; mouser (none) -> 81-GRM188R60J476ME5D; mouser2 (none) -> 81-ZRB18AR60J476ME1L; murata2 (none) -> ZRB18AR60J476ME01L
- HS1: FISCHER ELEKTRONIK 10037097 -> (none); fischer_elektronik (none) -> 10037097; fischer_elektronik_url (none) -> http://www.fischerelektronik.de/web_fischer/de_DE/K%C3%BChl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
- MK1, MK2: wegertseder (none) -> 2588-406; wegertseder_url (none) -> https://www.wegertseder.com/ArticleDetails.aspx?AKNUM=2588
- R1, R2, R3, R4: Vishay (none) -> CRCW06032K70FKEB; mouser (none) -> 71-CRCW06032K70FKEB
- U1, U2, U3, U4: mouser (none) -> 595-TLC5971RGER; texas instruments (none) -> TLC5971RGER
Changed lines of the file:
@@
 Title "LEDBoard 4x4 16bit"
 Date "2017-07-13"
-Rev "0.1"
+Rev "1.0"
 Comp "s-light.eu"
 Comment1 "designed by Stefan Krüger"
@@
 F 5 "https://www.reichelt.de/SMD-0603-von-1-bis-910-kOhm/SMD-0603-2-7K/3/index.html?ACTION=3&GROUPID=7968&ARTICLE=89435&OFFSET=100&" H 1150 2000 60  0001 C CNN "reichelt_url"
 F 6 "RC0603FR-072K7L" H 1150 2000 60  0001 C CNN "YAGEO"
+F 7 "CRCW06032K70FKEB" H 1150 2000 60  0001 C CNN "Vishay"
+F 8 "71-CRCW06032K70FKEB " H 0   0   60  0001 C CNN "mouser"
 	1    1150 2000
 	1    0    0    -1
@@
 F 5 "https://www.reichelt.de/Vielschicht-SMD-G0603/X7R-G0603-100N/3/index.html?ACTION=3&GROUPID=3166&ARTICLE=31873&OFFSET=100&" H 900 1400 60  0001 C CNN "reichelt_url"
 F 6 "CC0603KRX7R7BB104" H 900 1400 60  0001 C CNN "YAGEO"
+F 7 "81-GRM39X104K50D" H 0   0   60  0001 C CNN "mouser"
+F 8 "GRM188R71H104KA93D" H 0   0   60  0001 C CNN "murata"
 	1    900  1400
 	1    0    0    -1
@@
 F 1 "TLC5971RGER" H 2150 2900 50  0000 C CNN
 F 2 "Housings_DFN_QFN:Texas_S-PVQFN-N24_ThermalVias" H 1850 1550 20  0000 C CNN
-F 3 "" H 1800 2000 60  0000 C CNN
+F 3 "http://www.ti.com/product/TLC5971/description" H 1800 2000 60  0001 C CNN
+F 4 "595-TLC5971RGER" H 1850 2000 60  0001 C CNN "mouser"
+F 5 "TLC5971RGER" H 1850 2000 60  0001 C CNN "texas instruments"
 	1    1850 2000
 	1    0    0    -1
@@
 F 5 "https://www.reichelt.de/SMD-0603-von-1-bis-910-kOhm/SMD-0603-2-7K/3/index.html?ACTION=3&GROUPID=7968&ARTICLE=89435&OFFSET=100&" H 1150 2000 60  0001 C CNN "reichelt_url"
 F 6 "RC0603FR-072K7L" H 1150 2000 60  0001 C CNN "YAGEO"
+F 7 "CRCW06032K70FKEB" H 0   0   60  0001 C CNN "Vishay"
+F 8 "71-CRCW06032K70FKEB " H 0   0   60  0001 C CNN "mouser"
 	1    6450 2000
 	1    0    0    -1
@@
 F 5 "https://www.reichelt.de/Vielschicht-SMD-G0603/X7R-G0603-100N/3/index.html?ACTION=3&GROUPID=3166&ARTICLE=31873&OFFSET=100&" H 0   0   60  0001 C CNN "reichelt_url"
 F 6 "CC0603KRX7R7BB104" H 0   0   60  0001 C CNN "YAGEO"
+F 7 "81-GRM39X104K50D" H 0   0   60  0001 C CNN "mouser"
+F 8 "GRM188R71H104KA93D" H 0   0   60  0001 C CNN "murata"
 	1    6200 1400
 	1    0    0    -1
@@
 F 5 "https://www.reichelt.de/SMD-0603-von-1-bis-910-kOhm/SMD-0603-2-7K/3/index.html?ACTION=3&GROUPID=7968&ARTICLE=89435&OFFSET=100&" H 1150 2000 60  0001 C CNN "reichelt_url"
 F 6 "RC0603FR-072K7L" H 1150 2000 60  0001 C CNN "YAGEO"
+F 7 "CRCW06032K70FKEB" H 0   0   60  0001 C CNN "Vishay"
+F 8 "71-CRCW06032K70FKEB " H 0   0   60  0001 C CNN "mouser"
 	1    1150 4750
 	1    0    0    -1
@@
 F 5 "https://www.reichelt.de/Vielschicht-SMD-G0603/X7R-G0603-100N/3/index.html?ACTION=3&GROUPID=3166&ARTICLE=31873&OFFSET=100&" H 0   0   60  0001 C CNN "reichelt_url"
 F 6 "CC0603KRX7R7BB104" H 0   0   60  0001 C CNN "YAGEO"
+F 7 "81-GRM39X104K50D" H 0   0   60  0001 C CNN "mouser"
+F 8 "GRM188R71H104KA93D" H 0   0   60  0001 C CNN "murata"
 	1    900  4150
 	1    0    0    -1
@@
 F 2 "Housings_DFN_QFN:Texas_S-PVQFN-N24_ThermalVias" H 1850 4300 20  0000 C CNN
 F 3 "" H 1800 4750 60  0000 C CNN
+F 4 "595-TLC5971RGER" H 0   0   60  0001 C CNN "mouser"
+F 5 "TLC5971RGER" H 0   0   60  0001 C CNN "texas instruments"
 	1    1850 4750
 	1    0    0    -1
@@
 F 5 "https://www.reichelt.de/SMD-0603-von-1-bis-910-kOhm/SMD-0603-2-7K/3/index.html?ACTION=3&GROUPID=7968&ARTICLE=89435&OFFSET=100&" H 1150 2000 60  0001 C CNN "reichelt_url"
 F 6 "RC0603FR-072K7L" H 1150 2000 60  0001 C CNN "YAGEO"
+F 7 "CRCW06032K70FKEB" H 0   0   60  0001 C CNN "Vishay"
+F 8 "71-CRCW06032K70FKEB " H 0   0   60  0001 C CNN "mouser"
 	1    6450 4750
 	1    0    0    -1
@@
 F 5 "https://www.reichelt.de/Vielschicht-SMD-G0603/X7R-G0603-100N/3/index.html?ACTION=3&GROUPID=3166&ARTICLE=31873&OFFSET=100&" H 0   0   60  0001 C CNN "reichelt_url"
 F 6 "CC0603KRX7R7BB104" H 0   0   60  0001 C CNN "YAGEO"
+F 7 "81-GRM39X104K50D" H 0   0   60  0001 C CNN "mouser"
+F 8 "GRM188R71H104KA93D" H 0   0   60  0001 C CNN "murata"
 	1    6200 4150
 	1    0    0    -1
@@
 F 2 "Housings_DFN_QFN:Texas_S-PVQFN-N24_ThermalVias" H 7150 4300 20  0000 C CNN
 F 3 "" H 7100 4750 60  0000 C CNN
+F 4 "595-TLC5971RGER" H 0   0   60  0001 C CNN "mouser"
+F 5 "TLC5971RGER" H 0   0   60  0001 C CNN "texas instruments"
 	1    7150 4750
 	1    0    0    -1
@@
 F 2 "Housings_DFN_QFN:Texas_S-PVQFN-N24_ThermalVias" H 7150 1550 20  0000 C CNN
 F 3 "" H 7100 2000 60  0000 C CNN
+F 4 "595-TLC5971RGER" H 0   0   60  0001 C CNN "mouser"
+F 5 "TLC5971RGER" H 0   0   60  0001 C CNN "texas instruments"
 	1    7150 2000
 	1    0    0    -1
@@
 P 6050 7150
 F 0 "C5" H 6165 7196 50  0000 L CNN
-F 1 "47uF" H 6165 7105 50  0000 L CNN
+F 1 "47uF 6.3V" H 6165 7105 50  0000 L CNN
 F 2 "Capacitors_SMD:C_0603" H 6088 7000 50  0001 C CNN
 F 3 "" H 6050 7150 50  0001 C CNN
@@
 F 5 "https://www.reichelt.de/Vielschicht-SMD-G0603/X5R-G0603-47-6-3/3/index.html?ACTION=3&GROUPID=3166&ARTICLE=190489&OFFSET=100&" H 6050 7150 60  0001 C CNN "reichelt_url"
 F 6 "GRM188R60J476ME15D" H 6050 7150 60  0001 C CNN "murata"
+F 7 "ZRB18AR60J476ME01L" H 0   0   60  0001 C CNN "murata2"
+F 8 "81-GRM188R60J476ME5D" H 6050 7150 60  0001 C CNN "mouser"
+F 9 "81-ZRB18AR60J476ME1L " H 6050 7150 60  0001 C CNN "mouser2"
 	1    6050 7150
 	1    0    0    -1
@@
 F 2 "Mounting_Holes:MountingHole_3.2mm_M3_ISO7380_Pad" H 3950 6000 50  0001 C CNN
 F 3 "" H 3950 6000 50  0001 C CNN
+F 4 "2588-406" H 3950 6000 60  0001 C CNN "wegertseder"
+F 5 "https://www.wegertseder.com/ArticleDetails.aspx?AKNUM=2588" H 3950 6000 60  0001 C CNN "wegertseder_url"
 	1    3950 6000
 	1    0    0    -1
@@
 F 4 "V ICK PGA36X36" H 5650 6100 60  0001 C CNN "reichelt"
 F 5 "https://www.reichelt.de/Stiftkuehlkoerper/V-ICK-PGA36X36/3/index.html?ACTION=3&GROUPID=7773&ARTICLE=100978&OFFSET=100&" H 5650 6100 60  0001 C CNN "reichelt_url"
-F 6 "10037097" H 5650 6100 60  0001 C CNN "FISCHER ELEKTRONIK"
+F 6 "10037097" H 5650 6100 60  0001 C CNN "fischer_elektronik"
+F 7 "http://www.fischerelektronik.de/web_fischer/de_DE/K%C3%BChlk%C3%B6rper/B01/K%C3%BChlk%C3%B6rper%20f%C3%BCr%20PGA/PR/ICKPGA14x14x12_/$productCard/parameters/index.xhtml" H 5650 6100 60  0001 C CNN "fischer_elektronik_url"
 	1    5650 6100
 	1    0    0    -1
@@
 F 2 "Mounting_Holes:MountingHole_3.2mm_M3_ISO7380_Pad" H 4700 6000 50  0001 C CNN
 F 3 "" H 4700 6000 50  0001 C CNN
+F 4 "2588-406" H 4700 6000 60  0001 C CNN "wegertseder"
+F 5 "https://www.wegertseder.com/ArticleDetails.aspx?AKNUM=2588" H 4700 6000 60  0001 C CNN "wegertseder_url"
 	1    4700 6000
 	1    0    0    -1

Commit message: :memo: added missing part numbers mostly to get a consisten row count in the exported BOM csv file
Parts:
- J1, J6: reichelt (none) -> MPE 115-1-004
- J2: reichelt (none) -> MPE 115-1-006
Changed lines of the file:
@@
 F 2 "Socket_Strips:Socket_Strip_Straight_1x02_Pitch2.54mm" H 2350 7350 50  0001 C CNN
 F 3 "" H 2350 7350 50  0001 C CNN
+F 4 "MPE 115-1-004" H 2350 7250 60  0001 C CNN "reichelt"
 	1    2350 7250
 	1    0    0    -1
@@
 F 2 "Socket_Strips:Socket_Strip_Straight_1x02_Pitch2.54mm" H 1000 7350 50  0001 C CNN
 F 3 "" H 1000 7350 50  0001 C CNN
+F 4 "MPE 115-1-004" H 1000 7250 60  0001 C CNN "reichelt"
 	1    1000 7250
 	1    0    0    -1
@@
 F 2 "Socket_Strips:Socket_Strip_Straight_1x06_Pitch2.54mm" H 3950 7000 50  0001 C CNN
 F 3 "" H 3950 7000 50  0001 C CNN
+F 4 "MPE 115-1-006" H 3950 7000 60  0001 C CNN "reichelt"
 	1    3950 7000
 	-1   0    0    -1
