File: LEDBoard_4x4_16bit.sch (KiCad schematic (older format))
At the start: 35 parts, among them J1 signal_in, J2 power, J6 signal_out, U1 TLC5971RGER, U2 TLC5971RGER, U3 TLC5971RGER, U4 TLC5971RGER

Commit message: schematic: changed signal in & signal out to 3pin connector
Parts:
- J1: footprint Socket_Strips:Socket_Strip_Straight_1x02_Pitch2.54mm -> Socket_Strips:Socket_Strip_Straight_1x03_Pitch2.54mm; symbol CONN_01X02_MALE -> CONN_01X03; reichelt MPE 115-1-004 -> MPE 115-1-003
- J6: footprint Socket_Strips:Socket_Strip_Straight_1x02_Pitch2.54mm -> Socket_Strips:Socket_Strip_Straight_1x03_Pitch2.54mm; symbol CONN_01X02_FEMALE -> CONN_01X03; reichelt MPE 115-1-004 -> MPE 115-1-003
Connections:
- wire segments 84 -> 74
Changed lines of the file:
@@
 Sheet 1 1
 Title "LEDBoard 4x4 16bit"
-Date "2017-07-13"
-Rev "1.0"
+Date "03.08.2017"
+Rev "2.0.0"
 Comp "s-light.eu"
 Comment1 "designed by Stefan Krüger"
@@
 Text Label 1150 2700 2    60   ~ 0
 clock_in
-Text Label 1300 7150 0    60   ~ 0
+Text Label 1500 7050 0    60   ~ 0
 data_in
-Text Label 1300 7350 0    60   ~ 0
+Text Label 1500 7150 0    60   ~ 0
 clock_in
 Text Label 7850 2700 0    60   ~ 0
@@
 $EndComp
 $Comp
-L CONN_01X02_FEMALE J6
+L CONN_01X03 J6
 U 1 1 59685AEA
-P 2350 7250
-F 0 "J6" H 2350 7500 50  0000 L CNN
-F 1 "signal_out" V 2550 7050 50  0000 L CNN
-F 2 "Socket_Strips:Socket_Strip_Straight_1x02_Pitch2.54mm" H 2350 7350 50  0001 C CNN
-F 3 "" H 2350 7350 50  0001 C CNN
-F 4 "MPE 115-1-004" H 2350 7250 60  0001 C CNN "reichelt"
-	1    2350 7250
-	1    0    0    -1
-$EndComp
-$Comp
-L CONN_01X02_MALE J1
+P 2650 7150
+F 0 "J6" H 2600 7350 50  0000 L CNN
+F 1 "signal_out" V 2750 6950 50  0000 L CNN
+F 2 "Socket_Strips:Socket_Strip_Straight_1x03_Pitch2.54mm" H 2650 7250 50  0001 C CNN
+F 3 "" H 2650 7250 50  0001 C CNN
+F 4 "MPE 115-1-003" H 2650 7150 60  0001 C CNN "reichelt"
+	1    2650 7150
+	1    0    0    -1
+$EndComp
+$Comp
+L CONN_01X03 J1
 U 1 1 596860B5
-P 1000 7250
-F 0 "J1" H 950 7500 50  0000 C CNN
-F 1 "signal_in" V 800 7250 50  0000 C CNN
-F 2 "Socket_Strips:Socket_Strip_Straight_1x02_Pitch2.54mm" H 1000 7350 50  0001 C CNN
-F 3 "" H 1000 7350 50  0001 C CNN
-F 4 "MPE 115-1-004" H 1000 7250 60  0001 C CNN "reichelt"
-	1    1000 7250
-	1    0    0    -1
+P 1300 7150
+F 0 "J1" H 1300 7350 50  0000 C CNN
+F 1 "signal_in" V 1400 7150 50  0000 C CNN
+F 2 "Socket_Strips:Socket_Strip_Straight_1x03_Pitch2.54mm" H 1300 7250 50  0001 C CNN
+F 3 "" H 1300 7250 50  0001 C CNN
+F 4 "MPE 115-1-003" H 1300 7150 60  0001 C CNN "reichelt"
+	1    1300 7150
+	-1   0    0    -1
 $EndComp
 $Comp
@@
 	4150 7050 4350 7050
 Connection ~ 4350 7050
-Text Label 2250 7350 2    60   ~ 0
+Text Label 2450 7150 2    60   ~ 0
 clock_out
-Text Label 2250 7150 2    60   ~ 0
+Text Label 2450 7050 2    60   ~ 0
 data_out
 Text Label 7850 2600 0    60   ~ 0
@@
 Text Label 2550 5350 0    60   ~ 0
 data_2-3
-Wire Wire Line
-	1150 5350 650  5350
-Wire Wire Line
-	650  5350 650  3350
-Wire Wire Line
-	650  3350 8400 3350
-Wire Wire Line
-	8400 3350 8400 2600
-Wire Wire Line
-	8400 2600 7850 2600
-Wire Wire Line
-	5900 5350 6450 5350
-Wire Wire Line
-	5900 5600 5900 5350
-Wire Wire Line
-	3150 5600 5900 5600
-Wire Wire Line
-	3150 5350 3150 5600
-Wire Wire Line
-	2550 5350 3150 5350
+$Comp
+L GND #PWR047
+U 1 1 5982EC89
+P 2450 7250
+F 0 "#PWR047" H 2450 7000 50  0001 C CNN
+F 1 "GND" H 2455 7077 50  0000 C CNN
+F 2 "" H 2450 7250 50  0001 C CNN
+F 3 "" H 2450 7250 50  0001 C CNN
+	1    2450 7250
+	1    0    0    -1
+$EndComp
+$Comp
+L GND #PWR048
+U 1 1 5982F02C
+P 1500 7250
+F 0 "#PWR048" H 1500 7000 50  0001 C CNN
+F 1 "GND" H 1505 7077 50  0000 C CNN
+F 2 "" H 1500 7250 50  0001 C CNN
+F 3 "" H 1500 7250 50  0001 C CNN
+	1    1500 7250
+	1    0    0    -1
+$EndComp
+Text Label 6450 5350 2    60   ~ 0
+data_2-3
+Text Label 1150 5350 2    60   ~ 0
+data_1-2
 $EndSCHEMATC

Commit message: schematic: updated LED-Type to NSSM124D + generated BOM + exported NET-List + modified it (changed buggy nets)
Parts:
- D1.1, D1.2, D1.3, D1.4, D2.1, D2.2, D2.3, D2.4, D3.1, D3.2, D3.3, D3.4, D4.1, D4.2, D4.3, D4.4: footprint nichia:LED_NSSM032AT_wViaHeatSinkBig -> nichia:LED_NSSM124_wViaHeatSinkBig_LayoutCompatibleWithNSSM032AT; Nichia part NSSM032A -> NSSM124D
Changed lines of the file:
@@
 Sheet 1 1
 Title "LEDBoard 4x4 16bit"
-Date "03.08.2017"
-Rev "2.0.0"
+Date "08.08.2017"
+Rev "2.1.0"
 Comp "s-light.eu"
 Comment1 "designed by Stefan Krüger"
@@
 F 0 "D1.1" H 3950 2047 50  0000 C CNN
 F 1 "LED_1.1" H 3950 1956 50  0000 C CNN
-F 2 "nichia:LED_NSSM032AT_wViaHeatSinkBig" H 3950 1500 50  0001 C CNN
+F 2 "nichia:LED_NSSM124_wViaHeatSinkBig_LayoutCompatibleWithNSSM032AT" H 3950 1500 50  0001 C CNN
 F 3 "" H 3950 1500 50  0001 C CNN
-F 4 "NSSM032A" H 3950 1550 60  0001 C CNN "Nichia part"
+F 4 "NSSM124D" H 3950 1550 60  0001 C CNN "Nichia part"
 	1    3950 1550
 	1    0    0    -1
@@
 F 0 "D1.2" H 3950 2947 50  0000 C CNN
 F 1 "LED_1.2" H 3950 2856 50  0000 C CNN
-F 2 "nichia:LED_NSSM032AT_wViaHeatSinkBig" H 3950 2400 50  0001 C CNN
+F 2 "nichia:LED_NSSM124_wViaHeatSinkBig_LayoutCompatibleWithNSSM032AT" H 3950 2400 50  0001 C CNN
 F 3 "" H 3950 2400 50  0001 C CNN
-F 4 "NSSM032A" H 3950 2450 60  0001 C CNN "Nichia part"
+F 4 "NSSM124D" H 3950 2450 60  0001 C CNN "Nichia part"
 	1    3950 2450
 	1    0    0    -1
@@
 F 0 "D2.1" H 5150 2047 50  0000 C CNN
 F 1 "LED_2.1" H 5150 1956 50  0000 C CNN
-F 2 "nichia:LED_NSSM032AT_wViaHeatSinkBig" H 5150 1500 50  0001 C CNN
+F 2 "nichia:LED_NSSM124_wViaHeatSinkBig_LayoutCompatibleWithNSSM032AT" H 5150 1500 50  0001 C CNN
 F 3 "" H 5150 1500 50  0001 C CNN
-F 4 "NSSM032A" H 5150 1550 60  0001 C CNN "Nichia part"
+F 4 "NSSM124D" H 5150 1550 60  0001 C CNN "Nichia part"
 	1    5150 1550
 	1    0    0    -1
@@
 F 0 "D2.2" H 5150 2947 50  0000 C CNN
 F 1 "LED_2.2" H 5150 2856 50  0000 C CNN
-F 2 "nichia:LED_NSSM032AT_wViaHeatSinkBig" H 5150 2400 50  0001 C CNN
+F 2 "nichia:LED_NSSM124_wViaHeatSinkBig_LayoutCompatibleWithNSSM032AT" H 5150 2400 50  0001 C CNN
 F 3 "" H 5150 2400 50  0001 C CNN
-F 4 "NSSM032A" H 5150 2450 60  0001 C CNN "Nichia part"
+F 4 "NSSM124D" H 5150 2450 60  0001 C CNN "Nichia part"
 	1    5150 2450
 	1    0    0    -1
@@
 F 0 "D3.1" H 9250 2047 50  0000 C CNN
 F 1 "LED_3.1" H 9250 1956 50  0000 C CNN
-F 2 "nichia:LED_NSSM032AT_wViaHeatSinkBig" H 9250 1500 50  0001 C CNN
+F 2 "nichia:LED_NSSM124_wViaHeatSinkBig_LayoutCompatibleWithNSSM032AT" H 9250 1500 50  0001 C CNN
 F 3 "" H 9250 1500 50  0001 C CNN
-F 4 "NSSM032A" H 9250 1550 60  0001 C CNN "Nichia part"
+F 4 "NSSM124D" H 9250 1550 60  0001 C CNN "Nichia part"
 	1    9250 1550
 	1    0    0    -1
@@
 F 0 "D3.2" H 9250 2947 50  0000 C CNN
 F 1 "LED_3.2" H 9250 2856 50  0000 C CNN
-F 2 "nichia:LED_NSSM032AT_wViaHeatSinkBig" H 9250 2400 50  0001 C CNN
+F 2 "nichia:LED_NSSM124_wViaHeatSinkBig_LayoutCompatibleWithNSSM032AT" H 9250 2400 50  0001 C CNN
 F 3 "" H 9250 2400 50  0001 C CNN
-F 4 "NSSM032A" H 9250 2450 60  0001 C CNN "Nichia part"
+F 4 "NSSM124D" H 9250 2450 60  0001 C CNN "Nichia part"
 	1    9250 2450
 	1    0    0    -1
@@
 F 0 "D4.1" H 10450 2047 50  0000 C CNN
 F 1 "LED_4.1" H 10450 1956 50  0000 C CNN
-F 2 "nichia:LED_NSSM032AT_wViaHeatSinkBig" H 10450 1500 50  0001 C CNN
+F 2 "nichia:LED_NSSM124_wViaHeatSinkBig_LayoutCompatibleWithNSSM032AT" H 10450 1500 50  0001 C CNN
 F 3 "" H 10450 1500 50  0001 C CNN
-F 4 "NSSM032A" H 10450 1550 60  0001 C CNN "Nichia part"
+F 4 "NSSM124D" H 10450 1550 60  0001 C CNN "Nichia part"
 	1    10450 1550
 	1    0    0    -1
@@
 F 0 "D4.2" H 10450 2947 50  0000 C CNN
 F 1 "LED_4.2" H 10450 2856 50  0000 C CNN
-F 2 "nichia:LED_NSSM032AT_wViaHeatSinkBig" H 10450 2400 50  0001 C CNN
+F 2 "nichia:LED_NSSM124_wViaHeatSinkBig_LayoutCompatibleWithNSSM032AT" H 10450 2400 50  0001 C CNN
 F 3 "" H 10450 2400 50  0001 C CNN
-F 4 "NSSM032A" H 10450 2450 60  0001 C CNN "Nichia part"
+F 4 "NSSM124D" H 10450 2450 60  0001 C CNN "Nichia part"
 	1    10450 2450
 	1    0    0    -1
@@
 F 0 "D1.3" H 3950 4797 50  0000 C CNN
 F 1 "LED_1.3" H 3950 4706 50  0000 C CNN
-F 2 "nichia:LED_NSSM032AT_wViaHeatSinkBig" H 3950 4250 50  0001 C CNN
+F 2 "nichia:LED_NSSM124_wViaHeatSinkBig_LayoutCompatibleWithNSSM032AT" H 3950 4250 50  0001 C CNN
 F 3 "" H 3950 4250 50  0001 C CNN
-F 4 "NSSM032A" H 3950 4300 60  0001 C CNN "Nichia part"
+F 4 "NSSM124D" H 3950 4300 60  0001 C CNN "Nichia part"
 	1    3950 4300
 	1    0    0    -1
@@
 F 0 "D1.4" H 3950 5697 50  0000 C CNN
 F 1 "LED_1.4" H 3950 5606 50  0000 C CNN
-F 2 "nichia:LED_NSSM032AT_wViaHeatSinkBig" H 3950 5150 50  0001 C CNN
+F 2 "nichia:LED_NSSM124_wViaHeatSinkBig_LayoutCompatibleWithNSSM032AT" H 3950 5150 50  0001 C CNN
 F 3 "" H 3950 5150 50  0001 C CNN
-F 4 "NSSM032A" H 3950 5200 60  0001 C CNN "Nichia part"
+F 4 "NSSM124D" H 3950 5200 60  0001 C CNN "Nichia part"
 	1    3950 5200
 	1    0    0    -1
@@
 F 0 "D2.3" H 5150 4797 50  0000 C CNN
 F 1 "LED_2.3" H 5150 4706 50  0000 C CNN
-F 2 "nichia:LED_NSSM032AT_wViaHeatSinkBig" H 5150 4250 50  0001 C CNN
+F 2 "nichia:LED_NSSM124_wViaHeatSinkBig_LayoutCompatibleWithNSSM032AT" H 5150 4250 50  0001 C CNN
 F 3 "" H 5150 4250 50  0001 C CNN
-F 4 "NSSM032A" H 5150 4300 60  0001 C CNN "Nichia part"
+F 4 "NSSM124D" H 5150 4300 60  0001 C CNN "Nichia part"
 	1    5150 4300
 	1    0    0    -1
@@
 F 0 "D2.4" H 5150 5697 50  0000 C CNN
 F 1 "LED_2.4" H 5150 5606 50  0000 C CNN
-F 2 "nichia:LED_NSSM032AT_wViaHeatSinkBig" H 5150 5150 50  0001 C CNN
+F 2 "nichia:LED_NSSM124_wViaHeatSinkBig_LayoutCompatibleWithNSSM032AT" H 5150 5150 50  0001 C CNN
 F 3 "" H 5150 5150 50  0001 C CNN
-F 4 "NSSM032A" H 5150 5200 60  0001 C CNN "Nichia part"
+F 4 "NSSM124D" H 5150 5200 60  0001 C CNN "Nichia part"
 	1    5150 5200
 	1    0    0    -1
@@
 F 0 "D3.3" H 9250 4797 50  0000 C CNN
 F 1 "LED_3.3" H 9250 4706 50  0000 C CNN
-F 2 "nichia:LED_NSSM032AT_wViaHeatSinkBig" H 9250 4250 50  0001 C CNN
+F 2 "nichia:LED_NSSM124_wViaHeatSinkBig_LayoutCompatibleWithNSSM032AT" H 9250 4250 50  0001 C CNN
 F 3 "" H 9250 4250 50  0001 C CNN
-F 4 "NSSM032A" H 9250 4300 60  0001 C CNN "Nichia part"
+F 4 "NSSM124D" H 9250 4300 60  0001 C CNN "Nichia part"
 	1    9250 4300
 	1    0    0    -1
@@
 F 0 "D3.4" H 9250 5697 50  0000 C CNN
 F 1 "LED_3.4" H 9250 5606 50  0000 C CNN
-F 2 "nichia:LED_NSSM032AT_wViaHeatSinkBig" H 9250 5150 50  0001 C CNN
+F 2 "nichia:LED_NSSM124_wViaHeatSinkBig_LayoutCompatibleWithNSSM032AT" H 9250 5150 50  0001 C CNN
 F 3 "" H 9250 5150 50  0001 C CNN
-F 4 "NSSM032A" H 9250 5200 60  0001 C CNN "Nichia part"
+F 4 "NSSM124D" H 9250 5200 60  0001 C CNN "Nichia part"
 	1    9250 5200
 	1    0    0    -1
@@
 F 0 "D4.3" H 10450 4797 50  0000 C CNN
 F 1 "LED_4.3" H 10450 4706 50  0000 C CNN
-F 2 "nichia:LED_NSSM032AT_wViaHeatSinkBig" H 10450 4250 50  0001 C CNN
+F 2 "nichia:LED_NSSM124_wViaHeatSinkBig_LayoutCompatibleWithNSSM032AT" H 10450 4250 50  0001 C CNN
 F 3 "" H 10450 4250 50  0001 C CNN
-F 4 "NSSM032A" H 10450 4300 60  0001 C CNN "Nichia part"
+F 4 "NSSM124D" H 10450 4300 60  0001 C CNN "Nichia part"
 	1    10450 4300
 	1    0    0    -1
@@
 F 0 "D4.4" H 10450 5697 50  0000 C CNN
 F 1 "LED_4.4" H 10450 5606 50  0000 C CNN
-F 2 "nichia:LED_NSSM032AT_wViaHeatSinkBig" H 10450 5150 50  0001 C CNN
+F 2 "nichia:LED_NSSM124_wViaHeatSinkBig_LayoutCompatibleWithNSSM032AT" H 10450 5150 50  0001 C CNN
 F 3 "" H 10450 5150 50  0001 C CNN
-F 4 "NSSM032A" H 10450 5200 60  0001 C CNN "Nichia part"
+F 4 "NSSM124D" H 10450 5200 60  0001 C CNN "Nichia part"
 	1    10450 5200
 	1    0    0    -1

Commit message: started to do variant with TLC5971PWP --> HTSSOP housing
Parts:
- U1: value TLC5971RGER -> TLC5971PWPR; footprint Housings_DFN_QFN:Texas_S-PVQFN-N24_ThermalVias -> Housings_SSOP:HTSSOP-20-1EP_4.4x6.5mm_Pitch0.65mm_ThermalVias_TI_R-PDSO-G20; symbol TLC5971RGER -> TLC5971PWPR; mouser 595-TLC5971RGER -> 595-TLC5971PWPR; texas instruments TLC5971RGER -> TLC5971PWPR
Connections:
- net GND: now also U1.2 (GND), U1.21 (GND); no longer U1.18 (GND), U1.25 (GND)
- net LED_1.1_B: now also U1.5 (OUTB0); no longer U1.21 (OUTB0)
- net LED_1.1_G: now also U1.4 (OUTG0); no longer U1.20 (OUTG0)
- net LED_1.1_R: now also U1.3 (OUTR0); no longer U1.19 (OUTR0)
- net LED_1.2_B: now also U1.15 (OUTB2); no longer U1.9 (OUTB2)
- net LED_1.2_G: now also U1.14 (OUTG2); no longer U1.8 (OUTG2)
- net LED_1.2_R: now also U1.13 (OUTR2); no longer U1.7 (OUTR2)
- net LED_2.1_B: now also U1.8 (OUTB1); no longer U1.24 (OUTB1)
- net LED_2.1_G: now also U1.7 (OUTG1); no longer U1.23 (OUTG1)
- net LED_2.1_R: now also U1.6 (OUTR1); no longer U1.22 (OUTR1)
- net LED_2.2_B: now also U1.18 (OUTB3); no longer U1.12 (OUTB3)
- net LED_2.2_G: now also U1.17 (OUTG3); no longer U1.11 (OUTG3)
- net LED_2.2_R: now also U1.16 (OUTR3); no longer U1.10 (OUTR3)
- net U1_sense: now also U1.1 (IREF); no longer U1.16 (IREF)
- net VCC: now also U1.19 (VCC), U1.20 (VREG); no longer U1.13 (VCC), U1.15 (VREG)
- net clock_0-1: now also U1.11 (SCKO); no longer U1.5 (SCKO)
- net clock_in: now also U1.10 (SCKI); no longer U1.2 (SCKI)
- net data_0-1: now also U1.12 (SDTO); no longer U1.6 (SDTO)
- net data_in: now also U1.9 (SDTI); no longer U1.1 (SDTI)
Changed lines of the file:
@@
 $EndComp
 $Comp
-L TLC5971RGER U1
+L TLC5971PWPR U1
 U 1 1 596752BA
 P 1850 2000
 F 0 "U1" H 1950 3000 60  0000 C CNN
-F 1 "TLC5971RGER" H 2150 2900 50  0000 C CNN
-F 2 "Housings_DFN_QFN:Texas_S-PVQFN-N24_ThermalVias" H 1850 1550 20  0000 C CNN
+F 1 "TLC5971PWPR" H 2150 2900 50  0000 C CNN
+F 2 "Housings_SSOP:HTSSOP-20-1EP_4.4x6.5mm_Pitch0.65mm_ThermalVias_TI_R-PDSO-G20" H 1850 1550 20  0000 C CNN
 F 3 "http://www.ti.com/product/TLC5971/description" H 1800 2000 60  0001 C CNN
-F 4 "595-TLC5971RGER" H 1850 2000 60  0001 C CNN "mouser"
-F 5 "TLC5971RGER" H 1850 2000 60  0001 C CNN "texas instruments"
+F 4 "595-TLC5971PWPR" H 1850 2000 60  0001 C CNN "mouser"
+F 5 "TLC5971PWPR" H 1850 2000 60  0001 C CNN "texas instruments"
 	1    1850 2000
 	1    0    0    -1
