File: LEDBoard_4x4_16bit.sch (KiCad schematic (older format))
At the start: 35 parts, among them J1 signal_in, J2 power, J6 signal_out, U1 TLC5971PWPR, U2 TLC5971RGER, U3 TLC5971RGER, U4 TLC5971RGER

Commit message: preparation for new housings
Parts:
- D1.1, D1.2, D1.3, D1.4, D2.1, D2.2, D2.3, D2.4, D3.1, D3.2, D3.3, D3.4, D4.1, D4.2, D4.3, D4.4: footprint nichia:LED_NSSM124_wViaHeatSinkBig_LayoutCompatibleWithNSSM032AT -> nichia:LED_NSSM124_wViaHeatSinkBig
- U2, U3, U4: value TLC5971RGER -> TLC5971PWPR; footprint Housings_DFN_QFN:Texas_S-PVQFN-N24_ThermalVias -> Housings_SSOP:HTSSOP-20-1EP_4.4x6.5mm_Pitch0.65mm_ThermalVias_TI_R-PDSO-G20; symbol TLC5971RGER -> TLC5971PWPR; mouser 595-TLC5971RGER -> 595-TLC5971PWPR; texas instruments TLC5971RGER -> TLC5971PWPR
Connections:
- net GND: now also U2.2 (GND), U2.21 (GND), U3.2 (GND), U3.21 (GND), U4.2 (GND), U4.21 (GND); no longer U2.18 (GND), U2.25 (GND), U3.18 (GND), U3.25 (GND), U4.18 (GND), U4.25 (GND)
- net LED_1.3_B: now also U3.5 (OUTB0); no longer U3.21 (OUTB0)
- net LED_1.3_G: now also U3.4 (OUTG0); no longer U3.20 (OUTG0)
- net LED_1.3_R: now also U3.3 (OUTR0); no longer U3.19 (OUTR0)
- net LED_1.4_B: now also U3.15 (OUTB2); no longer U3.9 (OUTB2)
- net LED_1.4_G: now also U3.14 (OUTG2); no longer U3.8 (OUTG2)
- net LED_1.4_R: now also U3.13 (OUTR2); no longer U3.7 (OUTR2)
- net LED_2.3_B: now also U3.8 (OUTB1); no longer U3.24 (OUTB1)
- net LED_2.3_G: now also U3.7 (OUTG1); no longer U3.23 (OUTG1)
- net LED_2.3_R: now also U3.6 (OUTR1); no longer U3.22 (OUTR1)
- net LED_2.4_B: now also U3.18 (OUTB3); no longer U3.12 (OUTB3)
- net LED_2.4_G: now also U3.17 (OUTG3); no longer U3.11 (OUTG3)
- net LED_2.4_R: now also U3.16 (OUTR3); no longer U3.10 (OUTR3)
- net LED_3.1_B: now also U2.5 (OUTB0); no longer U2.21 (OUTB0)
- net LED_3.1_G: now also U2.4 (OUTG0); no longer U2.20 (OUTG0)
- net LED_3.1_R: now also U2.3 (OUTR0); no longer U2.19 (OUTR0)
- net LED_3.2_B: now also U2.15 (OUTB2); no longer U2.9 (OUTB2)
- net LED_3.2_G: now also U2.14 (OUTG2); no longer U2.8 (OUTG2)
- net LED_3.2_R: now also U2.13 (OUTR2); no longer U2.7 (OUTR2)
- net LED_3.3_B: now also U4.5 (OUTB0); no longer U4.21 (OUTB0)
- net LED_3.3_G: now also U4.4 (OUTG0); no longer U4.20 (OUTG0)
- net LED_3.3_R: now also U4.3 (OUTR0); no longer U4.19 (OUTR0)
- net LED_3.4_B: now also U4.15 (OUTB2); no longer U4.9 (OUTB2)
- net LED_3.4_G: now also U4.14 (OUTG2); no longer U4.8 (OUTG2)
- net LED_3.4_R: now also U4.13 (OUTR2); no longer U4.7 (OUTR2)
- net LED_4.1_B: now also U2.8 (OUTB1); no longer U2.24 (OUTB1)
- net LED_4.1_G: now also U2.7 (OUTG1); no longer U2.23 (OUTG1)
- net LED_4.1_R: now also U2.6 (OUTR1); no longer U2.22 (OUTR1)
- net LED_4.2_B: now also U2.18 (OUTB3); no longer U2.12 (OUTB3)
- net LED_4.2_G: now also U2.17 (OUTG3); no longer U2.11 (OUTG3)
- net LED_4.2_R: now also U2.16 (OUTR3); no longer U2.10 (OUTR3)
- net LED_4.3_B: now also U4.8 (OUTB1); no longer U4.24 (OUTB1)
- net LED_4.3_G: now also U4.7 (OUTG1); no longer U4.23 (OUTG1)
- net LED_4.3_R: now also U4.6 (OUTR1); no longer U4.22 (OUTR1)
- net LED_4.4_B: now also U4.18 (OUTB3); no longer U4.12 (OUTB3)
- net LED_4.4_G: now also U4.17 (OUTG3); no longer U4.11 (OUTG3)
- net LED_4.4_R: now also U4.16 (OUTR3); no longer U4.10 (OUTR3)
- net U2_sense: now also U2.1 (IREF); no longer U2.16 (IREF)
- net U3_sense: now also U3.1 (IREF); no longer U3.16 (IREF)
- net U4_sense: now also U4.1 (IREF); no longer U4.16 (IREF)
- net VCC: now also U2.19 (VCC), U2.20 (VREG), U3.19 (VCC), U3.20 (VREG), U4.19 (VCC), U4.20 (VREG); no longer U2.13 (VCC), U2.15 (VREG), U3.13 (VCC), U3.15 (VREG), U4.13 (VCC), U4.15 (VREG)
- net clock_0-1: now also U2.10 (SCKI); no longer U2.2 (SCKI)
- net clock_1-2: now also U2.11 (SCKO), U3.10 (SCKI); no longer U2.5 (SCKO), U3.2 (SCKI)
- net clock_2-3: now also U3.11 (SCKO), U4.10 (SCKI); no longer U3.5 (SCKO), U4.2 (SCKI)
- net clock_out: now also U4.11 (SCKO); no longer U4.5 (SCKO)
- net data_0-1: now also U2.9 (SDTI); no longer U2.1 (SDTI)
- net data_1-2: now also U2.12 (SDTO), U3.9 (SDTI); no longer U2.6 (SDTO), U3.1 (SDTI)
- net data_2-3: now also U3.12 (SDTO), U4.9 (SDTI); no longer U3.6 (SDTO), U4.1 (SDTI)
- net data_out: now also U4.12 (SDTO); no longer U4.6 (SDTO)
Changed lines of the file:
@@
 Sheet 1 1
 Title "LEDBoard 4x4 16bit"
-Date "08.08.2017"
-Rev "2.1.0"
+Date "31.08.2017"
+Rev "3.0.0"
 Comp "s-light.eu"
 Comment1 "designed by Stefan Krüger"
@@
 F 0 "D1.1" H 3950 2047 50  0000 C CNN
 F 1 "LED_1.1" H 3950 1956 50  0000 C CNN
-F 2 "nichia:LED_NSSM124_wViaHeatSinkBig_LayoutCompatibleWithNSSM032AT" H 3950 1500 50  0001 C CNN
+F 2 "nichia:LED_NSSM124_wViaHeatSinkBig" H 3950 1500 50  0001 C CNN
 F 3 "" H 3950 1500 50  0001 C CNN
 F 4 "NSSM124D" H 3950 1550 60  0001 C CNN "Nichia part"
@@
 F 0 "D1.2" H 3950 2947 50  0000 C CNN
 F 1 "LED_1.2" H 3950 2856 50  0000 C CNN
-F 2 "nichia:LED_NSSM124_wViaHeatSinkBig_LayoutCompatibleWithNSSM032AT" H 3950 2400 50  0001 C CNN
+F 2 "nichia:LED_NSSM124_wViaHeatSinkBig" H 3950 2400 50  0001 C CNN
 F 3 "" H 3950 2400 50  0001 C CNN
 F 4 "NSSM124D" H 3950 2450 60  0001 C CNN "Nichia part"
@@
 F 0 "D2.1" H 5150 2047 50  0000 C CNN
 F 1 "LED_2.1" H 5150 1956 50  0000 C CNN
-F 2 "nichia:LED_NSSM124_wViaHeatSinkBig_LayoutCompatibleWithNSSM032AT" H 5150 1500 50  0001 C CNN
+F 2 "nichia:LED_NSSM124_wViaHeatSinkBig" H 5150 1500 50  0001 C CNN
 F 3 "" H 5150 1500 50  0001 C CNN
 F 4 "NSSM124D" H 5150 1550 60  0001 C CNN "Nichia part"
@@
 F 0 "D2.2" H 5150 2947 50  0000 C CNN
 F 1 "LED_2.2" H 5150 2856 50  0000 C CNN
-F 2 "nichia:LED_NSSM124_wViaHeatSinkBig_LayoutCompatibleWithNSSM032AT" H 5150 2400 50  0001 C CNN
+F 2 "nichia:LED_NSSM124_wViaHeatSinkBig" H 5150 2400 50  0001 C CNN
 F 3 "" H 5150 2400 50  0001 C CNN
 F 4 "NSSM124D" H 5150 2450 60  0001 C CNN "Nichia part"
@@
 F 0 "D3.1" H 9250 2047 50  0000 C CNN
 F 1 "LED_3.1" H 9250 1956 50  0000 C CNN
-F 2 "nichia:LED_NSSM124_wViaHeatSinkBig_LayoutCompatibleWithNSSM032AT" H 9250 1500 50  0001 C CNN
+F 2 "nichia:LED_NSSM124_wViaHeatSinkBig" H 9250 1500 50  0001 C CNN
 F 3 "" H 9250 1500 50  0001 C CNN
 F 4 "NSSM124D" H 9250 1550 60  0001 C CNN "Nichia part"
@@
 F 0 "D3.2" H 9250 2947 50  0000 C CNN
 F 1 "LED_3.2" H 9250 2856 50  0000 C CNN
-F 2 "nichia:LED_NSSM124_wViaHeatSinkBig_LayoutCompatibleWithNSSM032AT" H 9250 2400 50  0001 C CNN
+F 2 "nichia:LED_NSSM124_wViaHeatSinkBig" H 9250 2400 50  0001 C CNN
 F 3 "" H 9250 2400 50  0001 C CNN
 F 4 "NSSM124D" H 9250 2450 60  0001 C CNN "Nichia part"
@@
 F 0 "D4.1" H 10450 2047 50  0000 C CNN
 F 1 "LED_4.1" H 10450 1956 50  0000 C CNN
-F 2 "nichia:LED_NSSM124_wViaHeatSinkBig_LayoutCompatibleWithNSSM032AT" H 10450 1500 50  0001 C CNN
+F 2 "nichia:LED_NSSM124_wViaHeatSinkBig" H 10450 1500 50  0001 C CNN
 F 3 "" H 10450 1500 50  0001 C CNN
 F 4 "NSSM124D" H 10450 1550 60  0001 C CNN "Nichia part"
@@
 F 0 "D4.2" H 10450 2947 50  0000 C CNN
 F 1 "LED_4.2" H 10450 2856 50  0000 C CNN
-F 2 "nichia:LED_NSSM124_wViaHeatSinkBig_LayoutCompatibleWithNSSM032AT" H 10450 2400 50  0001 C CNN
+F 2 "nichia:LED_NSSM124_wViaHeatSinkBig" H 10450 2400 50  0001 C CNN
 F 3 "" H 10450 2400 50  0001 C CNN
 F 4 "NSSM124D" H 10450 2450 60  0001 C CNN "Nichia part"
@@
 F 0 "D1.3" H 3950 4797 50  0000 C CNN
 F 1 "LED_1.3" H 3950 4706 50  0000 C CNN
-F 2 "nichia:LED_NSSM124_wViaHeatSinkBig_LayoutCompatibleWithNSSM032AT" H 3950 4250 50  0001 C CNN
+F 2 "nichia:LED_NSSM124_wViaHeatSinkBig" H 3950 4250 50  0001 C CNN
 F 3 "" H 3950 4250 50  0001 C CNN
 F 4 "NSSM124D" H 3950 4300 60  0001 C CNN "Nichia part"
@@
 $EndComp
 $Comp
-L TLC5971RGER U3
+L TLC5971PWPR U3
 U 1 1 59678C02
 P 1850 4750
 F 0 "U3" H 1950 5750 60  0000 C CNN
-F 1 "TLC5971RGER" H 2150 5650 50  0000 C CNN
-F 2 "Housings_DFN_QFN:Texas_S-PVQFN-N24_ThermalVias" H 1850 4300 20  0000 C CNN
+F 1 "TLC5971PWPR" H 2150 5650 50  0000 C CNN
+F 2 "Housings_SSOP:HTSSOP-20-1EP_4.4x6.5mm_Pitch0.65mm_ThermalVias_TI_R-PDSO-G20" H 1850 4300 20  0000 C CNN
 F 3 "" H 1800 4750 60  0000 C CNN
-F 4 "595-TLC5971RGER" H 0   0   60  0001 C CNN "mouser"
-F 5 "TLC5971RGER" H 0   0   60  0001 C CNN "texas instruments"
+F 4 "595-TLC5971PWPR" H 0   0   60  0001 C CNN "mouser"
+F 5 "TLC5971PWPR" H 0   0   60  0001 C CNN "texas instruments"
 	1    1850 4750
 	1    0    0    -1
@@
 F 0 "D1.4" H 3950 5697 50  0000 C CNN
 F 1 "LED_1.4" H 3950 5606 50  0000 C CNN
-F 2 "nichia:LED_NSSM124_wViaHeatSinkBig_LayoutCompatibleWithNSSM032AT" H 3950 5150 50  0001 C CNN
+F 2 "nichia:LED_NSSM124_wViaHeatSinkBig" H 3950 5150 50  0001 C CNN
 F 3 "" H 3950 5150 50  0001 C CNN
 F 4 "NSSM124D" H 3950 5200 60  0001 C CNN "Nichia part"
@@
 F 0 "D2.3" H 5150 4797 50  0000 C CNN
 F 1 "LED_2.3" H 5150 4706 50  0000 C CNN
-F 2 "nichia:LED_NSSM124_wViaHeatSinkBig_LayoutCompatibleWithNSSM032AT" H 5150 4250 50  0001 C CNN
+F 2 "nichia:LED_NSSM124_wViaHeatSinkBig" H 5150 4250 50  0001 C CNN
 F 3 "" H 5150 4250 50  0001 C CNN
 F 4 "NSSM124D" H 5150 4300 60  0001 C CNN "Nichia part"
@@
 F 0 "D2.4" H 5150 5697 50  0000 C CNN
 F 1 "LED_2.4" H 5150 5606 50  0000 C CNN
-F 2 "nichia:LED_NSSM124_wViaHeatSinkBig_LayoutCompatibleWithNSSM032AT" H 5150 5150 50  0001 C CNN
+F 2 "nichia:LED_NSSM124_wViaHeatSinkBig" H 5150 5150 50  0001 C CNN
 F 3 "" H 5150 5150 50  0001 C CNN
 F 4 "NSSM124D" H 5150 5200 60  0001 C CNN "Nichia part"
@@
 F 0 "D3.3" H 9250 4797 50  0000 C CNN
 F 1 "LED_3.3" H 9250 4706 50  0000 C CNN
-F 2 "nichia:LED_NSSM124_wViaHeatSinkBig_LayoutCompatibleWithNSSM032AT" H 9250 4250 50  0001 C CNN
+F 2 "nichia:LED_NSSM124_wViaHeatSinkBig" H 9250 4250 50  0001 C CNN
 F 3 "" H 9250 4250 50  0001 C CNN
 F 4 "NSSM124D" H 9250 4300 60  0001 C CNN "Nichia part"
@@
 $EndComp
 $Comp
-L TLC5971RGER U4
+L TLC5971PWPR U4
 U 1 1 59678C66
 P 7150 4750
 F 0 "U4" H 7250 5750 60  0000 C CNN
-F 1 "TLC5971RGER" H 7450 5650 50  0000 C CNN
-F 2 "Housings_DFN_QFN:Texas_S-PVQFN-N24_ThermalVias" H 7150 4300 20  0000 C CNN
+F 1 "TLC5971PWPR" H 7450 5650 50  0000 C CNN
+F 2 "Housings_SSOP:HTSSOP-20-1EP_4.4x6.5mm_Pitch0.65mm_ThermalVias_TI_R-PDSO-G20" H 7150 4300 20  0000 C CNN
 F 3 "" H 7100 4750 60  0000 C CNN
-F 4 "595-TLC5971RGER" H 0   0   60  0001 C CNN "mouser"
-F 5 "TLC5971RGER" H 0   0   60  0001 C CNN "texas instruments"
+F 4 "595-TLC5971PWPR" H 0   0   60  0001 C CNN "mouser"
+F 5 "TLC5971PWPR" H 0   0   60  0001 C CNN "texas instruments"
 	1    7150 4750
 	1    0    0    -1
@@
 F 0 "D3.4" H 9250 5697 50  0000 C CNN
 F 1 "LED_3.4" H 9250 5606 50  0000 C CNN
-F 2 "nichia:LED_NSSM124_wViaHeatSinkBig_LayoutCompatibleWithNSSM032AT" H 9250 5150 50  0001 C CNN
+F 2 "nichia:LED_NSSM124_wViaHeatSinkBig" H 9250 5150 50  0001 C CNN
 F 3 "" H 9250 5150 50  0001 C CNN
 F 4 "NSSM124D" H 9250 5200 60  0001 C CNN "Nichia part"
@@
 F 0 "D4.3" H 10450 4797 50  0000 C CNN
 F 1 "LED_4.3" H 10450 4706 50  0000 C CNN
-F 2 "nichia:LED_NSSM124_wViaHeatSinkBig_LayoutCompatibleWithNSSM032AT" H 10450 4250 50  0001 C CNN
+F 2 "nichia:LED_NSSM124_wViaHeatSinkBig" H 10450 4250 50  0001 C CNN
 F 3 "" H 10450 4250 50  0001 C CNN
 F 4 "NSSM124D" H 10450 4300 60  0001 C CNN "Nichia part"
@@
 F 0 "D4.4" H 10450 5697 50  0000 C CNN
 F 1 "LED_4.4" H 10450 5606 50  0000 C CNN
-F 2 "nichia:LED_NSSM124_wViaHeatSinkBig_LayoutCompatibleWithNSSM032AT" H 10450 5150 50  0001 C CNN
+F 2 "nichia:LED_NSSM124_wViaHeatSinkBig" H 10450 5150 50  0001 C CNN
 F 3 "" H 10450 5150 50  0001 C CNN
 F 4 "NSSM124D" H 10450 5200 60  0001 C CNN "Nichia part"
@@
 $EndComp
 $Comp
-L TLC5971RGER U2
+L TLC5971PWPR U2
 U 1 1 59677C50
 P 7150 2000
 F 0 "U2" H 7250 3000 60  0000 C CNN
-F 1 "TLC5971RGER" H 7450 2900 50  0000 C CNN
-F 2 "Housings_DFN_QFN:Texas_S-PVQFN-N24_ThermalVias" H 7150 1550 20  0000 C CNN
+F 1 "TLC5971PWPR" H 7450 2900 50  0000 C CNN
+F 2 "Housings_SSOP:HTSSOP-20-1EP_4.4x6.5mm_Pitch0.65mm_ThermalVias_TI_R-PDSO-G20" H 7150 1550 20  0000 C CNN
 F 3 "" H 7100 2000 60  0000 C CNN
-F 4 "595-TLC5971RGER" H 0   0   60  0001 C CNN "mouser"
-F 5 "TLC5971RGER" H 0   0   60  0001 C CNN "texas instruments"
+F 4 "595-TLC5971PWPR" H 0   0   60  0001 C CNN "mouser"
+F 5 "TLC5971PWPR" H 0   0   60  0001 C CNN "texas instruments"
 	1    7150 2000
 	1    0    0    -1

Commit message: updated BOM
Parts:
- D1.1, D1.2, D1.3, D1.4, D2.2, D2.3, D2.4, D3.1, D3.2, D3.3, D3.4, D4.1, D4.2, D4.3, D4.4: Lumitronix (none) -> 30201; Lumitronix_url (none) -> http://www.leds.de/Low-Mid-Power-LEDs/SMD-LEDs/Nichia-SMD-L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
- D2.1: Lumitronix (none) -> x; Lumitronix_url (none) -> xx
Changed lines of the file:
@@
 F 3 "" H 3950 1500 50  0001 C CNN
 F 4 "NSSM124D" H 3950 1550 60  0001 C CNN "Nichia part"
+F 5 "30201" H 3950 1550 60  0001 C CNN "Lumitronix"
+F 6 "http://www.leds.de/Low-Mid-Power-LEDs/SMD-LEDs/Nichia-SMD-LED-RGB-NSSM124DT.html" H 3950 1550 60  0001 C CNN "Lumitronix_url"
 	1    3950 1550
 	1    0    0    -1
@@
 F 3 "" H 3950 2400 50  0001 C CNN
 F 4 "NSSM124D" H 3950 2450 60  0001 C CNN "Nichia part"
+F 5 "30201" H 3950 2450 60  0001 C CNN "Lumitronix"
+F 6 "http://www.leds.de/Low-Mid-Power-LEDs/SMD-LEDs/Nichia-SMD-LED-RGB-NSSM124DT.html" H 3950 2450 60  0001 C CNN "Lumitronix_url"
 	1    3950 2450
 	1    0    0    -1
@@
 F 3 "" H 5150 1500 50  0001 C CNN
 F 4 "NSSM124D" H 5150 1550 60  0001 C CNN "Nichia part"
+F 5 "x" H 5150 1550 60  0001 C CNN "Lumitronix"
+F 6 "xx" H 5150 1550 60  0001 C CNN "Lumitronix_url"
 	1    5150 1550
 	1    0    0    -1
@@
 F 3 "" H 5150 2400 50  0001 C CNN
 F 4 "NSSM124D" H 5150 2450 60  0001 C CNN "Nichia part"
+F 5 "30201" H 5150 2450 60  0001 C CNN "Lumitronix"
+F 6 "http://www.leds.de/Low-Mid-Power-LEDs/SMD-LEDs/Nichia-SMD-LED-RGB-NSSM124DT.html" H 5150 2450 60  0001 C CNN "Lumitronix_url"
 	1    5150 2450
 	1    0    0    -1
@@
 F 3 "" H 9250 1500 50  0001 C CNN
 F 4 "NSSM124D" H 9250 1550 60  0001 C CNN "Nichia part"
+F 5 "30201" H 9250 1550 60  0001 C CNN "Lumitronix"
+F 6 "http://www.leds.de/Low-Mid-Power-LEDs/SMD-LEDs/Nichia-SMD-LED-RGB-NSSM124DT.html" H 9250 1550 60  0001 C CNN "Lumitronix_url"
 	1    9250 1550
 	1    0    0    -1
@@
 F 3 "" H 9250 2400 50  0001 C CNN
 F 4 "NSSM124D" H 9250 2450 60  0001 C CNN "Nichia part"
+F 5 "30201" H 9250 2450 60  0001 C CNN "Lumitronix"
+F 6 "http://www.leds.de/Low-Mid-Power-LEDs/SMD-LEDs/Nichia-SMD-LED-RGB-NSSM124DT.html" H 9250 2450 60  0001 C CNN "Lumitronix_url"
 	1    9250 2450
 	1    0    0    -1
@@
 F 3 "" H 10450 1500 50  0001 C CNN
 F 4 "NSSM124D" H 10450 1550 60  0001 C CNN "Nichia part"
+F 5 "30201" H 10450 1550 60  0001 C CNN "Lumitronix"
+F 6 "http://www.leds.de/Low-Mid-Power-LEDs/SMD-LEDs/Nichia-SMD-LED-RGB-NSSM124DT.html" H 10450 1550 60  0001 C CNN "Lumitronix_url"
 	1    10450 1550
 	1    0    0    -1
@@
 F 3 "" H 10450 2400 50  0001 C CNN
 F 4 "NSSM124D" H 10450 2450 60  0001 C CNN "Nichia part"
+F 5 "30201" H 10450 2450 60  0001 C CNN "Lumitronix"
+F 6 "http://www.leds.de/Low-Mid-Power-LEDs/SMD-LEDs/Nichia-SMD-LED-RGB-NSSM124DT.html" H 10450 2450 60  0001 C CNN "Lumitronix_url"
 	1    10450 2450
 	1    0    0    -1
@@
 F 3 "" H 3950 4250 50  0001 C CNN
 F 4 "NSSM124D" H 3950 4300 60  0001 C CNN "Nichia part"
+F 5 "30201" H 3950 4300 60  0001 C CNN "Lumitronix"
+F 6 "http://www.leds.de/Low-Mid-Power-LEDs/SMD-LEDs/Nichia-SMD-LED-RGB-NSSM124DT.html" H 3950 4300 60  0001 C CNN "Lumitronix_url"
 	1    3950 4300
 	1    0    0    -1
@@
 F 3 "" H 3950 5150 50  0001 C CNN
 F 4 "NSSM124D" H 3950 5200 60  0001 C CNN "Nichia part"
+F 5 "30201" H 3950 5200 60  0001 C CNN "Lumitronix"
+F 6 "http://www.leds.de/Low-Mid-Power-LEDs/SMD-LEDs/Nichia-SMD-LED-RGB-NSSM124DT.html" H 3950 5200 60  0001 C CNN "Lumitronix_url"
 	1    3950 5200
 	1    0    0    -1
@@
 F 3 "" H 5150 4250 50  0001 C CNN
 F 4 "NSSM124D" H 5150 4300 60  0001 C CNN "Nichia part"
+F 5 "30201" H 5150 4300 60  0001 C CNN "Lumitronix"
+F 6 "http://www.leds.de/Low-Mid-Power-LEDs/SMD-LEDs/Nichia-SMD-LED-RGB-NSSM124DT.html" H 5150 4300 60  0001 C CNN "Lumitronix_url"
 	1    5150 4300
 	1    0    0    -1
@@
 F 3 "" H 5150 5150 50  0001 C CNN
 F 4 "NSSM124D" H 5150 5200 60  0001 C CNN "Nichia part"
+F 5 "30201" H 5150 5200 60  0001 C CNN "Lumitronix"
+F 6 "http://www.leds.de/Low-Mid-Power-LEDs/SMD-LEDs/Nichia-SMD-LED-RGB-NSSM124DT.html" H 5150 5200 60  0001 C CNN "Lumitronix_url"
 	1    5150 5200
 	1    0    0    -1
@@
 F 3 "" H 9250 4250 50  0001 C CNN
 F 4 "NSSM124D" H 9250 4300 60  0001 C CNN "Nichia part"
+F 5 "30201" H 9250 4300 60  0001 C CNN "Lumitronix"
+F 6 "http://www.leds.de/Low-Mid-Power-LEDs/SMD-LEDs/Nichia-SMD-LED-RGB-NSSM124DT.html" H 9250 4300 60  0001 C CNN "Lumitronix_url"
 	1    9250 4300
 	1    0    0    -1
@@
 F 3 "" H 9250 5150 50  0001 C CNN
 F 4 "NSSM124D" H 9250 5200 60  0001 C CNN "Nichia part"
+F 5 "30201" H 9250 5200 60  0001 C CNN "Lumitronix"
+F 6 "http://www.leds.de/Low-Mid-Power-LEDs/SMD-LEDs/Nichia-SMD-LED-RGB-NSSM124DT.html" H 9250 5200 60  0001 C CNN "Lumitronix_url"
 	1    9250 5200
 	1    0    0    -1
@@
 F 3 "" H 10450 4250 50  0001 C CNN
 F 4 "NSSM124D" H 10450 4300 60  0001 C CNN "Nichia part"
+F 5 "30201" H 10450 4300 60  0001 C CNN "Lumitronix"
+F 6 "http://www.leds.de/Low-Mid-Power-LEDs/SMD-LEDs/Nichia-SMD-LED-RGB-NSSM124DT.html" H 10450 4300 60  0001 C CNN "Lumitronix_url"
 	1    10450 4300
 	1    0    0    -1
@@
 F 3 "" H 10450 5150 50  0001 C CNN
 F 4 "NSSM124D" H 10450 5200 60  0001 C CNN "Nichia part"
+F 5 "30201" H 10450 5200 60  0001 C CNN "Lumitronix"
+F 6 "http://www.leds.de/Low-Mid-Power-LEDs/SMD-LEDs/Nichia-SMD-LED-RGB-NSSM124DT.html" H 10450 5200 60  0001 C CNN "Lumitronix_url"
 	1    10450 5200
 	1    0    0    -1

Commit message: updated exports and images
Parts:
- D2.1: Lumitronix x -> 30201; Lumitronix_url xx -> http://www.leds.de/Low-Mid-Power-LEDs/SMD-LEDs/Nichia-SMD-L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
Changed lines of the file:
@@
 F 3 "" H 5150 1500 50  0001 C CNN
 F 4 "NSSM124D" H 5150 1550 60  0001 C CNN "Nichia part"
-F 5 "x" H 5150 1550 60  0001 C CNN "Lumitronix"
-F 6 "xx" H 5150 1550 60  0001 C CNN "Lumitronix_url"
+F 5 "30201" H 5150 1550 60  0001 C CNN "Lumitronix"
+F 6 "http://www.leds.de/Low-Mid-Power-LEDs/SMD-LEDs/Nichia-SMD-LED-RGB-NSSM124DT.html" H 5150 1550 60  0001 C CNN "Lumitronix_url"
 	1    5150 1550
 	1    0    0    -1
