File: LEDBoard_4x4_16bit.sch (KiCad schematic (older format))
At the start: 35 parts, among them J1 signal_in, J2 power, J6 signal_out, U1 TLC5971PWPR, U2 TLC5971PWPR, U3 TLC5971PWPR, U4 TLC5971PWPR

Commit message: updated Resistors and Capacitors for easier handsoldering
Parts:
- C1, C2, C3, C4, C5: footprint Capacitors_SMD:C_0603 -> Capacitors_SMD:C_0603_HandSoldering
- R1, R2, R3, R4: footprint Resistors_SMD:R_0603 -> Resistors_SMD:R_0603_HandSoldering
Changed lines of the file:
@@
 Sheet 1 1
 Title "LEDBoard 4x4 16bit"
-Date "27.09.2017"
-Rev "3.0.1"
+Date "16.12.2017"
+Rev "3.0.2"
 Comp "s-light.eu"
 Comment1 "designed by Stefan Krüger"
@@
 F 0 "R1" H 1220 2046 50  0000 L CNN
 F 1 "2k7 1%" H 1220 1955 50  0000 L CNN
-F 2 "Resistors_SMD:R_0603" V 1080 2000 50  0001 C CNN
+F 2 "Resistors_SMD:R_0603_HandSoldering" V 1080 2000 50  0001 C CNN
 F 3 "" H 1150 2000 50  0001 C CNN
 F 4 "SMD-0603 2,7K" H 1150 2000 60  0001 C CNN "reichelt"
@@
 F 0 "C1" H 1015 1446 50  0000 L CNN
 F 1 "100nF" H 1015 1355 50  0000 L CNN
-F 2 "Capacitors_SMD:C_0603" H 938 1250 50  0001 C CNN
+F 2 "Capacitors_SMD:C_0603_HandSoldering" H 938 1250 50  0001 C CNN
 F 3 "" H 900 1400 50  0001 C CNN
 F 4 "X7R-G0603 100N" H 900 1400 60  0001 C CNN "reichelt"
@@
 F 0 "R2" H 6520 2046 50  0000 L CNN
 F 1 "2k7 1%" H 6520 1955 50  0000 L CNN
-F 2 "Resistors_SMD:R_0603" V 6380 2000 50  0001 C CNN
+F 2 "Resistors_SMD:R_0603_HandSoldering" V 6380 2000 50  0001 C CNN
 F 3 "" H 6450 2000 50  0001 C CNN
 F 4 "SMD-0603 2,7K" H 1150 2000 60  0001 C CNN "reichelt"
@@
 F 0 "C2" H 6315 1446 50  0000 L CNN
 F 1 "100nF" H 6315 1355 50  0000 L CNN
-F 2 "Capacitors_SMD:C_0603" H 6238 1250 50  0001 C CNN
+F 2 "Capacitors_SMD:C_0603_HandSoldering" H 6238 1250 50  0001 C CNN
 F 3 "" H 6200 1400 50  0001 C CNN
 F 4 "X7R-G0603 100N" H 0   0   60  0001 C CNN "reichelt"
@@
 F 0 "R3" H 1220 4796 50  0000 L CNN
 F 1 "2k7 1%" H 1220 4705 50  0000 L CNN
-F 2 "Resistors_SMD:R_0603" V 1080 4750 50  0001 C CNN
+F 2 "Resistors_SMD:R_0603_HandSoldering" V 1080 4750 50  0001 C CNN
 F 3 "" H 1150 4750 50  0001 C CNN
 F 4 "SMD-0603 2,7K" H 1150 2000 60  0001 C CNN "reichelt"
@@
 F 0 "C3" H 1015 4196 50  0000 L CNN
 F 1 "100nF" H 1015 4105 50  0000 L CNN
-F 2 "Capacitors_SMD:C_0603" H 938 4000 50  0001 C CNN
+F 2 "Capacitors_SMD:C_0603_HandSoldering" H 938 4000 50  0001 C CNN
 F 3 "" H 900 4150 50  0001 C CNN
 F 4 "X7R-G0603 100N" H 0   0   60  0001 C CNN "reichelt"
@@
 F 0 "R4" H 6520 4796 50  0000 L CNN
 F 1 "2k7 1%" H 6520 4705 50  0000 L CNN
-F 2 "Resistors_SMD:R_0603" V 6380 4750 50  0001 C CNN
+F 2 "Resistors_SMD:R_0603_HandSoldering" V 6380 4750 50  0001 C CNN
 F 3 "" H 6450 4750 50  0001 C CNN
 F 4 "SMD-0603 2,7K" H 1150 2000 60  0001 C CNN "reichelt"
@@
 F 0 "C4" H 6315 4196 50  0000 L CNN
 F 1 "100nF" H 6315 4105 50  0000 L CNN
-F 2 "Capacitors_SMD:C_0603" H 6238 4000 50  0001 C CNN
+F 2 "Capacitors_SMD:C_0603_HandSoldering" H 6238 4000 50  0001 C CNN
 F 3 "" H 6200 4150 50  0001 C CNN
 F 4 "X7R-G0603 100N" H 0   0   60  0001 C CNN "reichelt"
@@
 F 0 "C5" H 6165 7196 50  0000 L CNN
 F 1 "47uF 6.3V" H 6165 7105 50  0000 L CNN
-F 2 "Capacitors_SMD:C_0603" H 6088 7000 50  0001 C CNN
+F 2 "Capacitors_SMD:C_0603_HandSoldering" H 6088 7000 50  0001 C CNN
 F 3 "" H 6050 7150 50  0001 C CNN
 F 4 "X5R-G0603 47/6,3" H 6050 7150 60  0001 C CNN "reichelt"
